File: hardware/key_module/key_module.kicad_sch (KiCad schematic)
At the start: 0 parts

Commit message: Remove brain board project and consolidate into key_module
Parts:
- added C1: 100nF, Capacitor_Tantalum_SMD:CP_EIA-2012-12_Kemet-R_HandSolder, symbol Device:C
- added C2: 4.7uF, Capacitor_Tantalum_SMD:CP_EIA-2012-12_Kemet-R_HandSolder, symbol Device:C
- added C3, C4: 10uF, Capacitor_Tantalum_SMD:CP_EIA-2012-12_Kemet-R_HandSolder, symbol Device:C_Polarized
- added D1, D10, D11, D12, D13, D14, D15, D16, D2, D3, D4, D5, D6, D7, D8, D9: SK6812MINI, LED_SMD:LED_SK6812MINI_PLCC4_3.5x3.5mm_P1.75mm, symbol LED:SK6812MINI
- added J1: SWD, Connector_PinHeader_2.54mm:PinHeader_1x04_P2.54mm_Vertical, symbol Connector_Generic:Conn_01x04
- added J2: WEST, Connector_PinHeader_2.54mm:PinHeader_1x06_P2.54mm_Horizontal, symbol Connector_Generic:Conn_01x04
- added J5: EAST, Connector_PinSocket_2.54mm:PinSocket_1x06_P2.54mm_Horizontal, symbol Connector_Generic:Conn_01x04
- added U1: STM32G030F6Px, Package_SO:TSSOP-20_4.4x6.5mm_P0.65mm, symbol MCU_ST_STM32G0:STM32G030F6Px
- added U10, U11, U12, U13, U14, U15, U16, U17, U18, U19, U4, U5, U6, U7, U8, U9: ~, hexis:HE, symbol hexis:HE
- added U2, U3: TMUX1308DYYR, 4ms_Package_SOT:SOT-23-THIN-16, symbol 4ms_IC:TMUX1308DYYR
- added U20: AMS1117-3.3, Package_TO_SOT_SMD:SOT-223-3_TabPin2, symbol Regulator_Linear:AMS1117-3.3
Connections:
- new net: D10.1 (DOUT), D11.3 (DIN)
- new net: D10.3 (DIN), D9.1 (DOUT)
- new net: D8.1 (DOUT), D9.3 (DIN)
- new net: D7.1 (DOUT), D8.3 (DIN)
- new net: D6.1 (DOUT), D7.3 (DIN)
- new net: D4.1 (DOUT), D5.3 (DIN)
- new net: D3.1 (DOUT), D4.3 (DIN)
- new net: D5.1 (DOUT), D6.3 (DIN)
- new net: D2.1 (DOUT), D3.3 (DIN)
- new net: D1.1 (DOUT), D2.3 (DIN)
- new net: D13.1 (DOUT), D14.3 (DIN)
- new net: D12.1 (DOUT), D13.3 (DIN)
- new net: D15.1 (DOUT), D16.3 (DIN)
- new net: D11.1 (DOUT), D12.3 (DIN)
- new net: D14.1 (DOUT), D15.3 (DIN)
- new net +3.3V: C1.1, C2.1, C4.1, J1.1 (Pin_1), U1.4 (VDD), U10.1 (VCC), U11.1 (VCC), U12.1 (VCC), U13.1 (VCC), U14.1 (VCC), U15.1 (VCC), U16.1 (VCC), U17.1 (VCC), U18.1 (VCC), U19.1 (VCC), U2.16 (VDD), U20.2 (VO), U3.16 (VDD), U4.1 (VCC), U5.1 (VCC), U6.1 (VCC), U7.1 (VCC), U8.1 (VCC), U9.1 (VCC)
- new net +5V: C3.1, D1.4 (VDD), D10.4 (VDD), D11.4 (VDD), D12.4 (VDD), D13.4 (VDD), D14.4 (VDD), D15.4 (VDD), D16.4 (VDD), D2.4 (VDD), D3.4 (VDD), D4.4 (VDD), D5.4 (VDD), D6.4 (VDD), D7.4 (VDD), D8.4 (VDD), D9.4 (VDD), J2.1 (Pin_1), J5.1 (Pin_1), U20.3 (VI)
- new net GND: C1.2, C2.2, C3.2, C4.2, D1.2 (VSS), D10.2 (VSS), D11.2 (VSS), D12.2 (VSS), D13.2 (VSS), D14.2 (VSS), D15.2 (VSS), D16.2 (VSS), D2.2 (VSS), D3.2 (VSS), D4.2 (VSS), D5.2 (VSS), D6.2 (VSS), D7.2 (VSS), D8.2 (VSS), D9.2 (VSS), J1.4 (Pin_4), J2.4 (Pin_4), J5.4 (Pin_4), U1.5 (VSS), U10.3 (GND), U11.3 (GND), U12.3 (GND), U13.3 (GND), U14.3 (GND), U15.3 (GND), U16.3 (GND), U17.3 (GND), U18.3 (GND), U19.3 (GND), U2.6 (/EN), U2.8 (GND), U20.1 (GND), U3.6 (/EN), U3.8 (GND), U4.3 (GND), U5.3 (GND), U6.3 (GND), U7.3 (GND), U8.3 (GND), U9.3 (GND)
- new net I2C_SCL: J2.2 (Pin_2), J5.2 (Pin_2), U1.16 (PA9/PA11)
- new net I2C_SDA: J2.3 (Pin_3), J5.3 (Pin_3), U1.17 (PA10/PA12)
- new net MCU_LED: D1.3 (DIN), U1.12 (PA5)
- new net S1: U2.13 (S0), U4.2 (OUT)
- new net S10: U13.2 (OUT), U3.14 (S1)
- new net S11: U14.2 (OUT), U3.15 (S2)
- new net S12: U15.2 (OUT), U3.12 (S3)
- new net S13: U16.2 (OUT), U3.1 (S4)
- new net S14: U17.2 (OUT), U3.5 (S5)
- new net S15: U18.2 (OUT), U3.2 (S6)
- new net S16: U19.2 (OUT), U3.4 (S7)
- new net S2: U2.14 (S1), U5.2 (OUT)
- new net S3: U2.15 (S2), U6.2 (OUT)
- new net S4: U2.12 (S3), U7.2 (OUT)
- new net S5: U2.1 (S4), U8.2 (OUT)
- new net S6: U2.5 (S5), U9.2 (OUT)
- new net S7: U10.2 (OUT), U2.2 (S6)
- new net S8: U11.2 (OUT), U2.4 (S7)
- new net S9: U12.2 (OUT), U3.13 (S0)
- new net SWCLK: J1.3 (Pin_3), U1.19 (PA14/PA15)
- new net SWDIO: J1.2 (Pin_2), U1.18 (PA13)
- new net TMUX1_OUT: U1.7 (PA0), U2.3 (D)
- new net TMUX2_OUT: U1.8 (PA1), U3.3 (D)
- new net TMUX_A0: U1.9 (PA2), U2.11 (A0), U3.11 (A0)
- new net TMUX_A1: U1.10 (PA3), U2.10 (A1), U3.10 (A1)
- new net TMUX_A2: U1.11 (PA4), U2.9 (A2), U3.9 (A2)
- no-connect marks 0 -> 1
